Commit message: Add files via upload
Pan joint problem is fixed

File: phantomx_pincher_robot_arm_edited/urdf/phantomx_pincher_robot_arm_edited.urdf (robot description, URDF)
Before this commit: robot phantomx_pincher_robot_arm_edited, 8 links, 7 joints
Links:
- link base_link: mass 0 -> 0.12375
- link right_gripper_link: mass 0.00650667742243692 -> 0.00650667742243691
Joints:
- joint arm_shoulder_pan_joint: type fixed -> continuous
