Commit message: Arm stl is updated

File: urdf/phantomx_pincher_robot_arm_edited.urdf (robot description, URDF)
Before this commit: robot phantomx_pincher_robot_arm_edited, 8 links, 7 joints
Links:
- link arm_elbow_flex_link: mass 0.0599991472451478 -> 0.059999
- link arm_shoulder_lift_link: mass 0.0599991472451477 -> 0.059999
- link arm_shoulder_pan_link: mass 0.0435262757095505 -> 0.043526
- link arm_wrist_flex_link: mass 0.0513446164144625 -> 0.051345
- link left_gripper_link: mass 0.00650667742243691 -> 0.00650667742243688
Joints:
- joint arm_elbow_flex_joint: axis 0 1 0 -> 0 -1 0; origin xyz=0 0 -0.107 rpy=0 0 3.1416 -> xyz=0 0 0.107 rpy=2.7756E-15 0 0
- joint arm_shoulder_lift_joint: origin xyz=0 0 0.0415 rpy=-3.1416 1.0749E-13 -1.4901E-08 -> xyz=0 0 0.0415 rpy=0 0 0
- joint arm_shoulder_pan_joint: origin xyz=-0.034767 -0.2961 0.089775 rpy=-7.2132E-06 -6.1215E-17 -1.5708 -> xyz=-0.034767 -0.2961 0.089775 rpy=-6.123E-17 0 0
- joint arm_wrist_flex_joint: axis 0 1 0 -> 0 -1 0; origin xyz=0 0 -0.107 rpy=0 0 0 -> xyz=0 0 0.107 rpy=-2.7756E-15 0 0
- joint arm_wrist_revol_joint: origin xyz=-0.00025427 0.0014125 -0.06645 rpy=3.1416 0 1.5708 -> xyz=-0.00025427 0.006 0.06645 rpy=0 -1.1102E-14 3.1416
- joint left_gripper_joint: limit lower=0 upper=0.015 effort=0 velocity=0 -> effort=0 velocity=0; origin xyz=0.00015 -0.014476 0.042144 rpy=0 0 0 -> xyz=0.00015 -0.015611 0.042144 rpy=-5.5511E-15 0 6.163E-29
- joint right_gripper_joint: axis 0 1 0 -> 0 -1 0; limit lower=0 upper=0.015 effort=0 velocity=0 -> effort=0 velocity=0; origin xyz=0.00015 0.013982 0.042144 rpy=0 0 3.1416 -> xyz=0.00015 0.015117 0.042144 rpy=0 -1.1102E-14 3.1416
